File: pcb_0222/pcb_0222.kicad_sch (KiCad schematic)
At the start: 52 parts

Commit message: Schematic On Review
Parts:
- removed C?: 4.7uF, passives_smd:C_1206_h1.8mm, symbol C_capacitors_ceramic:C_1206_4.7uF_50V_X7R
- removed C? (x2): 100nF, passives_smd:C_0603, symbol C_capacitors_ceramic:C_0603_100nF_50V
- removed C?: 1pF, passives_smd:C_0603, symbol C_capacitors_ceramic:C_0603_1pF_50V
- removed J?: SM08B-PASS-TBT, symbol J_connectors_headers:SM08B-PASS-TBT
- removed J?: SM02B-PASS-TBT, symbol J_connectors_headers:SM02B-PASS-TBT
- removed L?: 12uH, symbol L_inductors:L_6.8x6.8mm_12uH_1.7A
- removed R?: 200K, passives_smd:R_0603, symbol R_resistors:R_0603_200K_1%
- removed R?: 2.2K, passives_smd:R_1206, symbol R_resistors:R_1206_2K7_1%_500mW
- removed R?: 22.1K, passives_smd:R_0603, symbol R_resistors:R_0603_22.1K_1%
- removed R?: 1K, symbol R_resistors:R_2512_1K_1%_1W_AEC_Q200
- removed R?: 2.87M, passives_smd:R_0603, symbol R_resistors:R_0603_2.87M_1%
- removed R?: 0R, passives_smd:R_0603, symbol R_resistors:R_0603_0R
- removed R?: 10K, passives_smd:R_0603, symbol R_resistors:R_0603_10K_1%
- removed TP?: (no value), testpoints:TP_SMD_2mm, symbol TP_testpoints:TP_SMD_2MM
- added C10, C11, C12: 100nF, passives_smd:C_0603, symbol C_capacitors_ceramic:C_0603_100nF_50V
- added C13: 4.7uF, passives_smd:C_0603, symbol C_capacitors_ceramic:C_0603_4.7uF_10V
- added C2: 1pF, passives_smd:C_0603, symbol C_capacitors_ceramic:C_0603_1pF_50V_C0G
- added C3: 4.7uF, passives_smd:C_0603, symbol C_capacitors_ceramic:C_0603_4.7uF_35V
- added C7, C8: 10nF, passives_smd:C_0603, symbol C_capacitors_ceramic:C_0603_10nF_50V
- added J2: SM02B-PASS-TBT, symbol J_connectors_headers:SM02B-PASS-TBT
- added J4: HEADER_MALE_THT_0.1"_2x1, connectors_headers:77311-118-02LF, symbol J_connectors_headers:HEADER_MALE_THT_0.1{dblquote}_2x1
- added J5, J8: HEADER_MALE_THT_0.1"_4x1, symbol J_connectors_headers:HEADER_MALE_THT_0.1{dblquote}_4x1
- added J6: SM08B-PASS-TBT, symbol J_connectors_headers:SM08B-PASS-TBT
- added J7: TC-2030-IDC, symbol J_connectors_prog:TC-2030-IDC
- added L1: 12uH, symbol L_inductors:L_44.88mm3_6.8x6.8mm_12uH_1.7A
- added PB1: (no value), switches_smd:7914J-1-000, symbol S_switches_pushbutton:7914J-1-000
- added R1: 0R, passives_smd:R_0603, symbol R_resistors:R_0603_0R
- added R16: 10K, passives_smd:R_0603, symbol R_resistors:R_0603_10K_1%
- added R21, R22: 4K7, passives_smd:R_0603, symbol R_resistors:R_0603_4K7_1%
- added R3: 2.2K, passives_smd:R_1206, symbol R_resistors:R_1206_2.2K_0.5W
- added R4: 2.87M, passives_smd:R_0603, symbol R_resistors:R_0603_2.87M_1%_0.1W
- added R5: 22.1K, passives_smd:R_0603, symbol R_resistors:R_0603_22.1K_1%
- added R7: 1K, passives_smd:R_2512, symbol R_resistors:R_2512_1K_1%_1W_AEC-Q200
- added R8: 200K, passives_smd:R_0603, symbol R_resistors:R_0603_200K_1%_0.1W
- added TP1, TP10, TP11, TP12, TP13, TP14, TP15, TP17, TP4, TP5, TP6, TP7, TP8, TP9: (no value), testpoints:TP_SMD_2mm, symbol TP_testpoints:TP_SMD_2MM
- added U3: STM32C011F6P6, symbol U_microcontrollers:STM32C011F6P6
- C1, C4, C6: renamed from C?; TEMP. COEFF. (none) -> X7R; TOLERANCE (none) -> 10%; VOLTAGE (none) -> 50V
- R18, R19, R6: renamed from R?; PWR (none) -> 1/10W; TEMP. COEFF. (none) -> ±100ppm/°C; TOLERANCE (none) -> 1%
- gave numbers to parts that had none: 31
Connections:
- net +3V3: now also C10.2, C12.2, C13.2, J4.1, J5.1, J7.1 (VREF), J8.1, R16.2, R21.2, R22.2, TP14.1, TP15.1, U3.4 (VDD/VDDA)
- net FB: now also C2.1, R5.1
- net GND: now also C10.1, C11.1, C12.1, C13.1, C3.1, C7.1, C8.1, J2.2, J5.4, J7. (GND), J8.4, PB1.1, PB1.2, R7.1, R8.1, TP12.1, TP13.1, U3.5 (VSS/VSSA)
- net MCU_BCD0: now also TP4.1, U3.11 (PA4)
- net MCU_BCD1: now also TP8.1, U3.12 (PA5)
- net MCU_BCD2: now also TP10.1, U3.13 (PA6)
- net MCU_BCD3: now also TP11.1, U3.14 (PA7)
- net MCU_DIP1: now also TP7.1, U3.2 (PC14-OSCX_IN)
- net MCU_DIP2: now also TP9.1, U3.3 (PC15-OSCX_OUT)
- net MCU_SW1: now also C8.2, TP6.1, U3.9 (PA2)
- net MCU_SW2: now also C7.2, J2.1, R16.1, TP5.1, U3.10 (PA3)
- net SW: now also L1.1
- net VB_IP: now also J6.1, J6.3, J6.5, J6.7, R1.1, R3.2, TP1.1; no longer TP2.1
- net at C6.2, Q1.1, U1.A: now also R7.2
- net at C9.1, K1.9 (COM_2): now also J6.2, J6.4, J6.6, J6.8
- net at U2.4 (EN): now also R4.1, R8.2
- net at C5.2, R2.1, R6.2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: now also C2.2, L1.2, R5.2
- net at LED1.A: now also R3.1
- net at C4.2, U2.5 (VIN): now also TP2.1, C3.2, R1.2, R4.2
- net UC_LED renamed MCU_LED
- net MCU_LED: now also U3.8 (PA1)
- net UC_RELAY renamed MCU_RELAY
- net MCU_RELAY: now also TP17.1, U3.7 (PA0)
- new net NRST: C11.2, J7.6 (NRST), PB1.3, PB1.4, U3.6 (PF2-NRST)
- new net RX1: J5.3, U3.17 (PA12[PA10])
- new net SCL1: J8.3, R21.1, U3.1 (PB7)
- new net SDA1: J8.2, R22.1, U3.20 (PB6)
- new net SWCLK: J4.2, J7.3 (SWCLK), U3.19 (PA14-BOOT0)
- new net SWDIO: J7.2 (SWDIO), U3.18 (PA13)
- new net TX1: J5.2, U3.16 (PA11[PA9])
- no-connect marks 3 -> 6
Other:
- note added: "(Internal Rpu)"
- note added: "MCU"
- note added: "VREF provided by BOARD"
- note removed: "Auxiliary"
- moved on the sheet: C1, C4, C5, C6, C9, D1, J1, J3, K1, LED1, Q1, Q2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

Commit message: Footprints On Review
Parts:
- removed Q1: BSP170P, symbol Q_transistors_pmos:BSP170P
- removed S2: MRSSV1DR10SMGWTR, symbol S_switches_rotary:MRSSV1DR10SMGWTR
- added Q1: BSP170PH6327XTSA1, packages_smd:SOT-223-4, symbol Q_transistors_pmos:BSP170PH6327XTSA1
- added S2: 1-1825013-0, switches_smd:1-1825013-0, symbol S_switches_rotary:1-1825013-0
- J1: footprint (none) -> connectors_terminal_blocks:5442206
- J2, J3: footprint (none) -> connectors_headers:SM02B-PASS-TBT
- J5, J8: footprint (none) -> connectors_headers:61300411121
- J6: footprint (none) -> connectors_headers:SM08B-PASS-TBT
- J7: footprint (none) -> connectors_prog:TC2030-IDC
- K1: footprint (none) -> relays:EE23NUH
- L1: footprint (none) -> passives_smd:L_44.88mm3_6.8x6.8mm_Bourns_SRR6038-120Y
- Q2: footprint (none) -> packages_smd:SOT-23-3
- S1: footprint (none) -> switches_smd:DS04-254-2-02BK-SMT-TR
- U1: value NZH5V1B -> NZH5V1B,115; footprint (none) -> diodes_smd:SOD-123F
- U2: footprint (none) -> packages_smd:SOT-23-6
- U3: footprint (none) -> packages_smd:TSSOP-20 [6.4x4.4x1.2,P=0.65]mm
- renumbered LED4 to LED3, LED3 to LED4, R19 to R18, R18 to R19
Connections:
- net GND: now also S2.C1, S2.C2
- net MCU_BCD0: now also S2.1
- net MCU_BCD1: now also S2.2
- net MCU_BCD2: now also S2.4
- net MCU_BCD3: now also S2.8
- net VB_IP: now also Q1.3 (S)
- net at C6.2, R7.2, U1.A: now also Q1.1
- net at F1.1, TVS1.C: now also Q1.2 (D), Q1.4 (D)

Commit message: Placement on Review
Parts:
- added M1, M2, M3, M4: (no value), mechanical:mounting_hole_M3_NPTH, symbol M_mechanical:mounting_hole_M3_NPTH
- added TP18: (no value), testpoints:TP_SMD_0.8mm, symbol TP_testpoints:TP_SMD_2MM
- C5: DIGIKEY_PN_CT (none) -> 490-GRM188Z71A106MA73JCT-ND; MANUFACTURER (none) -> Murata Electronics; TEMP. COEFF. (none) -> X7R; TOLERANCE (none) -> 20%; VOLTAGE (none) -> 10V
- F1: DIGIKEY_PN_CT (none) -> 5923-0ZCF0100AF2ACT-ND; MANUFACTURER (none) -> Bel Fuse Inc.
- LED3: footprint passives_smd:R_0603 -> leds_smd:LED_0603
- LED4: DIGIKEY_PN_CT (none) -> 160-1436-1-ND; MANUFACTURER (none) -> Lite-On Inc.; PARTNO LTST-C190KSKT -> LTST-C190KRKT
- TP1, TP10, TP11, TP16, TP17, TP2, TP3, TP4, TP5, TP6, TP7, TP8, TP9: footprint testpoints:TP_SMD_2mm -> testpoints:TP_SMD_0.8mm
Connections:
- net GND: now also J1.2, J7.4 (GND); no longer J1.1, J7. (GND)
- net VB: now also J1.1; no longer J1.2
- net at R4.1, R8.2, U2.4 (EN): now also TP18.1
Other:
- moved on the sheet: J1, R18, R4, R8

Commit message: Placement on Review
Parts:
- added C14: 10uF, passives_smd:C_1210_TDK_CGA6_2.8mm_Tall, symbol C_capacitors_ceramic:C_1210_10uF_75V_X7R_AECQ200
- added J9: SM08B-PASS-TBT, connectors_headers:SM08B-PASS-TBT, symbol J_connectors_headers:SM08B-PASS-TBT
Connections:
- net GND: now also J1.1, K1.5 (NO_1); no longer J1.2
- net VB: now also J1.2; no longer J1.1
- net VB_IP: now also C14.2, J9.1, J9.3, J9.5, J9.7
- net at K1.4 (COM_1): now also C14.1, J9.2, J9.4, J9.6, J9.8
- no-connect marks 6 -> 4
Other:
- note added: "4 pairs (Power + GND) to drive 4 LED strips"
- note removed: "Route 4 pairs (Power + GND) to drive 4 LED strips"
- moved on the sheet: C7, C8, C9, D1, J2, J3, J6, K1, LED3, LED4, Q2, R10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

Commit message: Working on SCH review
Parts:
- removed J8: HEADER_MALE_THT_0.1"_4x1, connectors_headers:61300411121, symbol J_connectors_headers:HEADER_MALE_THT_0.1{dblquote}_4x1
- removed R21: 4K7, passives_smd:R_0603, symbol R_resistors:R_0603_4K7_1%
- removed R5: 22.1K, passives_smd:R_0603, symbol R_resistors:R_0603_22.1K_1%
- removed R9: 69.8K, passives_smd:R_0603, symbol R_resistors:R_0603_69.8K_1%
- removed U1: NZH5V1B,115, diodes_smd:SOD-123F, symbol D_diodes_zener:NZH5V1B
- added C8: 10nF, passives_smd:C_0603, symbol C_capacitors_ceramic:C_0603_10nF_50V
- added D1: NZH5V1B,115, diodes_smd:SOD-123F, symbol D_diodes_zener:NZH5V1B
- added J9: HEADER_MALE_THT_0.1"_4x1, connectors_headers:61300411121, symbol J_connectors_headers:HEADER_MALE_THT_0.1{dblquote}_4x1
- added R14: 10K, passives_smd:R_0603, symbol R_resistors:R_0603_10K_1%
- added R23: 4K7, passives_smd:R_0603, symbol R_resistors:R_0603_4K7_1%
- added R5: 69.8K, passives_smd:R_0603, symbol R_resistors:R_0603_69.8K_1%
- added R9: 22.1K, passives_smd:R_0603, symbol R_resistors:R_0603_22.1K_1%
- added TP10: (no value), testpoints:TP_SMD_0.8mm, symbol TP_testpoints:TP_SMD_2MM
- added TVS2, TVS3, TVS4, TVS6: 3V3, symbol D_diodes_tvs:SP1103C-01UTG
- added TVS5, TVS7, TVS8: USBLC6-2SC6, packages_smd:SOT-23-6 [2.8x2.93x1.1,P=0.95]mm, symbol D_diodes_tvs:USBLC6-2SC6
- C10: renamed from C8; POPULATE DNP -> (none)
- C9: renamed from C7; POPULATE DNP -> (none)
- J1: DIGIKEY_PN_CT (none) -> 277-12547-ND; MANUFACTURER (none) -> Phoenix Contact
- J7: renamed from J5; POPULATE DNP -> (none); now not fitted
- J8: renamed from J4; POPULATE DNP -> (none); now not fitted
- K1, Q1, Q2: CRITICAL (none) -> TRUE
- R22: POPULATE DNP -> (none); now not fitted
- TVS1: DIGIKEY_PN_CT (none) -> 18-SMAJ26CACT-ND; MANUFACTURER (none) -> Littelfuse Inc.
- U1: renamed from U2; CRITICAL (none) -> TRUE
- U2: renamed from U3; CRITICAL (none) -> TRUE
- renumbered C10 to C11, C9 to C12, C11 to C13, C12 to C14, C13 to C15, C14 to C7, D1 to D2, J9 to J4, J7 to J5, R16 to R15, R17 to R16, R14 to R17, R15 to R18, R18 to R20, R20 to R21, TP12 to TP1, TP5 to TP11, TP6 to TP12, TP8 to TP13, TP7 to TP14, TP10 to TP15, TP9 to TP16, TP11 to TP17, TP16 to TP18, TP17 to TP19, TP13 to TP2, TP14 to TP3, TP15 to TP4, TP1 to TP5, TP2 to TP6, TP3 to TP7, TP18 to TP8, TP4 to TP9
Connections:
- net +3V3: now also J9.1, R14.2, R23.2, TVS5.5 (VBUS), TVS7.5 (VBUS), TVS8.5 (VBUS)
- net FB: now also R5.1, R9.2
- net GND: now also PB1.3, PB1.4, C8.1, J9.4, R9.1, TVS2.A, TVS3.A, TVS4.A, TVS5.2 (GND), TVS6.A, TVS7.2 (GND), TVS8.2 (GND); no longer PB1.1, PB1.2
- net MCU_SW1: now also TVS4.C
- net MCU_SW2: now also TVS3.C
- net NRST: now also TVS6.C; no longer PB1.3, PB1.4
- net RX1: now also TVS7.4 (I/O2); no longer J7.3
- net SCL1: now also R23.1, TVS8.4 (I/O2)
- net SDA1: now also TVS8.6 (I/O1)
- net SWCLK: now also TVS5.4 (I/O2); no longer J5.3 (SWCLK)
- net SWDIO: now also TVS5.6 (I/O1); no longer J5.2 (SWDIO)
- net TX1: now also TVS7.6 (I/O1); no longer J7.2
- net VB_IP: now also D1.C
- net at C2.2, C5.2, L1.2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: now also R5.2
- net at C6.2, Q1.1, R7.2: now also D1.A
- net MCU_TEST: now reaches U2.15 (PA8)
- net MCU_TEST: now also PB1.1, PB1.2, C8.2, R14.1, TP10.1, TVS2.C
- new net: J5.2 (SWDIO), TVS5.1 (I/O1)
- new net: J5.3 (SWCLK), TVS5.3 (I/O2)
- new net: J7.2, TVS7.1 (I/O1)
- new net: J7.3, TVS7.3 (I/O2)
- new net: J9.2, TVS8.1 (I/O1)
- new net: J9.3, TVS8.3 (I/O2)
- no-connect marks 4 -> 3
Other:
- moved on the sheet: C1, C10, C11, C12, C13, C14, C15, C2, C3, C4, C5, C6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

Commit message: SCH review comments fixed
Parts:
- removed C15: 4.7uF, passives_smd:C_0603, symbol C_capacitors_ceramic:C_0603_4.7uF_10V
- added C15: 4.7uF, passives_smd:C_0603, symbol C_capacitors_ceramic:C_0603_4.7uF_35V
- C1, C11, C13, C14, C4, C6: DIGIKEY_PN_CT (none) -> 399-C0603C104K5RACTUCT-ND; MANUFACTURER (none) -> KEMET
- C10, C8, C9: DIGIKEY_PN_CT (none) -> 478-KGM15AR71H103KTCT-ND; MANUFACTURER (none) -> KYOCERA AVX
- C12, C7: MANUFACTURER (none) -> TDK; Manufacturer TDK -> (none)
- C2: DIGIKEY_PN_CT (none) -> 478-KGM15ACG1H1R0CT-ND; MANUFACTURER (none) -> KYOCERA AVX
- C3: DIGIKEY_PN_CT (none) -> 490-7205-1-ND; MANUFACTURER (none) -> Murata Electronics
- D1: DIGIKEY_PN_CT (none) -> 1727-NZH5V1B,115CT-ND; MANUFACTURER (none) -> Nexperia USA Inc.
- D2: DIGIKEY_PN_CT (none) -> 5399-B5819WCT-ND; MANUFACTURER (none) -> Shenzhen Slkormicro Semicon Co., Ltd.
- J2, J3: DIGIKEY_PN_CT (none) -> 455-SM02B-PASS-TBTCT-ND; MANUFACTURER (none) -> JST Sales America Inc.
- J4, J6: DIGIKEY_PN_CT (none) -> 455-SM08B-PASS-TBTCT-ND; MANUFACTURER (none) -> JST Sales America Inc.
- J5: DIGIKEY_PN_CT (none) -> TC2030-IDC-ND; MANUFACTURER Tag-Connect -> Tag-Connect LLC
- J8: DIGIKEY_PN_CT (none) -> 609-4434-ND; MANUFACTURER (none) -> Amphenol ICC (FCI)
- K1: DIGIKEY_PN_CT (none) -> 399-EE2-3NUH-ND; MANUFACTURER (none) -> KEMET
- L1: DIGIKEY_PN_CT (none) -> SRR6038-120YCT-ND; MANUFACTURER (none) -> Bourns Inc.
- LED1, LED2: CRITICAL NO -> (none); DIGIKEY_PN_CT (none) -> 160-LTST-C190GKTCT-ND; MANUFACTURER (none) -> Lite-On Inc.
- LED3: DIGIKEY_PN_CT (none) -> 160-1437-1-ND; MANUFACTURER (none) -> Lite-On Inc.
- PB1: DIGIKEY_PN_CT (none) -> 7914J-1-000-ND; MANUFACTURER (none) -> Bourns Inc.
- Q1: DIGIKEY_PN_CT (none) -> BSP170PH6327XTSA1CT-ND; MANUFACTURER (none) -> Infineon Technologies
- Q2: CRITICAL TRUE -> (none); MANUFACTURER (none) -> Shenzhen Slkormicro Semicon Co., Ltd.
- R1, R2: DIGIKEY_PN_CT (none) -> RMCF0603ZT0R00CT-ND; MANUFACTURER (none) -> Stackpole Electronics Inc
- R10, R11, R12, R13, R14, R15, R16, R17, R18: DIGIKEY_PN_CT (none) -> 311-10.0KHRCT-ND; MANUFACTURER (none) -> YAGEO
- R19, R20, R6: DIGIKEY_PN_CT (none) -> 13-RC0603FR-13120RLCT-ND; MANUFACTURER (none) -> YAGEO
- R21: DIGIKEY_PN_CT (none) -> RMCF0603FT1K00CT-ND; MANUFACTURER (none) -> Stackpole Electronics Inc
- R22, R23: DIGIKEY_PN_CT (none) -> P4.70KHCT-ND; MANUFACTURER (none) -> Panasonic Industry
- R3: DIGIKEY_PN_CT (none) -> 1712-CRGH1206F2K2CT-ND; MANUFACTURER (none) -> TE Connectivity Passive Product
- R4: DIGIKEY_PN_CT (none) -> 541-2.87MHCT-ND; MANUFACTURER (none) -> Vishay Dale
- R5: DIGIKEY_PN_CT (none) -> 311-69.8KHRCT-ND; MANUFACTURER (none) -> YAGEO; PWR (none) -> 0.1W; TEMP. COEFF. (none) -> ±100ppm/°C; TOLERANCE (none) -> 1%
- R7: DIGIKEY_PN_CT (none) -> 541-1.00KAFCT-ND; MANUFACTURER (none) -> Vishay Dale
- R8: DIGIKEY_PN_CT (none) -> 541-200KHCT-ND; MANUFACTURER (none) -> Vishay Dale
- R9: DIGIKEY_PN_CT (none) -> 311-22.1KHRCT-ND; MANUFACTURER (none) -> YAGEO; PWR (none) -> 0.1W; TEMP. COEFF. (none) -> ±100ppm/°C; TOLERANCE (none) -> 1%
- S1: DIGIKEY_PN_CT (none) -> 2223-DS04-254-2-02BK-SMT-CT-ND; MANUFACTURER (none) -> Same Sky (Formerly CUI Devices)
- S2: DIGIKEY_PN_CT (none) -> 2266-1-1825013-0-ND; MANUFACTURER (none) -> TE Connectivity ALCOSWITCH Switches
- TVS2, TVS3, TVS4, TVS6: footprint (none) -> diodes_smd:2-DFN_(1.6x1)
- TVS5, TVS7, TVS8: DIGIKEY_PN_CT (none) -> 497-5235-1-ND; MANUFACTURER (none) -> STMicroelectronics
- U1: DIGIKEY_PN_CT (none) -> 296-LMR54406DBVRCT-ND; MANUFACTURER (none) -> Texas Instruments
- U2: DIGIKEY_PN_CT (none) -> 497-STM32C011F6P6-ND; MANUFACTURER (none) -> STMicroelectronics
Connections:
- net +3V3: now also C15.2
- net GND: now also C15.1
Other:
- moved on the sheet: C10, C8, C9, TVS2, TVS3, TVS4

Commit message: working on Layout
Parts:
- removed J1: 5442206, connectors_terminal_blocks:5442206, symbol J_connectors_terminal_blocks:5442206
- added J1: S2P-VH, connectors_headers:S2P-VH, symbol J_connectors_headers:S2P-VH
Connections:
- net GND: now also J1.1
- net VB: now also J1.2
