File: pcb_0222/pcb_0222.kicad_sch (KiCad schematic)
At the start: 94 parts, among them J1 S2P-VH, J2 SM02B-PASS-TBT, J3 SM02B-PASS-TBT, J4 SM08B-PASS-TBT, J5 TC-2030-IDC, J6 SM08B-PASS-TBT, J7 HEADER_MALE_THT_0.1"_4x1, J8 HEADER_MALE_THT_0.1"_2x1, J9 HEADER_MALE_THT_0.1"_4x1, K1 EE2-3NUH, Q1 BSP170PH6327XTSA1, Q2 BC817-16, U1 LMR54406DBVR, U2 STM32C011F6P6

Commit message: Layout Review Pending + Preliminary Manufacturer Package Generated
Parts:
- J7, J9: DIGIKEY_PN_CT (none) -> 732-5317-ND; MANUFACTURER (none) -> Würth Elektronik
Changed lines of the file:
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@@
 			)
 		)
+		(property "MANUFACTURER" "Würth Elektronik"
+			(at 152.4 185.42 0)
+			(hide yes)
+			(show_name no)
+			(do_not_autoplace no)
+			(effects
+				(font
+					(size 1.27 1.27)
+				)
+			)
+		)
+		(property "DIGIKEY_PN_CT" "732-5317-ND"
+			(at 152.4 185.42 0)
+			(hide yes)
+			(show_name no)
+			(do_not_autoplace no)
+			(effects
+				(font
+					(size 1.27 1.27)
+				)
+			)
+		)
 		(pin "4"
 		)
@@
 			(at 152.4 161.29 0)
 			(hide yes)
+			(show_name no)
+			(do_not_autoplace no)
+			(effects
+				(font
+					(size 1.27 1.27)
+				)
+			)
+		)
+		(property "MANUFACTURER" "Würth Elektronik"
+			(at 152.4 161.29 0)
+			(hide yes)
+			(show_name no)
+			(do_not_autoplace no)
+			(effects
+				(font
+					(size 1.27 1.27)
+				)
+			)
+		)
+		(property "DIGIKEY_PN_CT" "732-5317-ND"
+			(at 152.4 161.29 0)
+			(hide yes)

Commit message: C7, C12 PARTNO upsated + LED4 VALUE updated + S2 MPN changed to CD10RM0SB
Parts:
- removed S2: 1-1825013-0, switches_smd:1-1825013-0, symbol S_switches_rotary:1-1825013-0
- added S2: CD10RM0SB, switches_smd:CD10RM0SB, symbol S_switches_rotary:CD10RM0SB
- C12, C7: PARTNO GRT188R61H105KE13D -> CGA6P1X7R1N106K250AC
- LED4: value LTST-C190KSKT -> LTST-C190KRKT
Connections:
- net GND: now also S2.C1, S2.C2
- net MCU_BCD0: now also S2.1
- net MCU_BCD1: now also S2.2
- net MCU_BCD2: now also S2.4
- net MCU_BCD3: now also S2.8
Changed lines of the file:
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@@
 	)
 	(junction
+		(at 87.63 93.98)
+		(diameter 0)
+		(color 0 0 0 0)
+	)
+	(junction
 		(at 34.29 31.75)
 		(diameter 1.27)
@@
 	)
 	(junction
-		(at 87.63 93.98)
-		(diameter 0)
-		(color 0 0 0 0)
-	)
-	(junction
 		(at 113.03 54.61)
 		(diameter 0)
@@
 	(wire
 		(pts
-			(xy 87.63 96.52) (xy 87.63 93.98)
+			(xy 87.63 95.25) (xy 87.63 93.98)
 		)
 		(stroke
@@
 		)
 	)
-	(label "MCU_BCD3"
-		(at 31.75 97.79 0)
-		(effects
-			(font
-				(size 1.27 1.27)
-				(color 0 0 255 1)
-			)
-			(justify left bottom)
-		)
-	)
 	(label "MCU_SW1"
 		(at 91.44 125.73 180)
@@
 		)
 	)
-	(label "MCU_BCD0"
-		(at 31.75 86.36 0)
+	(label "MCU_BCD3"
+		(at 31.75 97.79 0)
 		(effects
 			(font
@@
 		)
 	)
+	(label "MCU_BCD0"
+		(at 31.75 86.36 0)
+		(effects
+			(font
+				(size 1.27 1.27)
+				(color 0 0 255 1)
+			)
+			(justify left bottom)
+		)
+	)
 	(label "SDA1"
 		(at 101.6 177.8 0)
@@
 			)
 		)
-		(property "PARTNO" "GRT188R61H105KE13D"
+		(property "PARTNO" "CGA6P1X7R1N106K250AC"
 			(at 246.38 127 0)
 			(hide yes)
@@
 			)
 		)
-		(property "Description" "10 µF ±10% 75V Ceramic Capacitor X7R 1210 (3225 Metric) AEC-Q200"
+		(property "Description" "10 µF ±10% 75V Ceramic Capacitor X7R 1210"
 			(at 247.65 78.74 0)
 			(hide yes)
@@
 			)
 		)
-		(property "PARTNO" "GRT188R61H105KE13D"
+		(property "PARTNO" "CGA6P1X7R1N106K250AC"
 			(at 247.65 78.74 0)
 			(hide yes)
@@
 			)
 		)
-		(property "Value" "LTST-C190KSKT"
+		(property "Value" "LTST-C190KRKT"
 			(at 203.2 128.2699 0)
 			(hide yes)
@@
 	(symbol
 		(lib_id "power:GND")
-		(at 87.63 96.52 0)
+		(at 87.63 95.25 0)
 		(unit 1)
 		(body_style 1)
@@
 		(dnp no)
 		(property "Reference" "#PWR017"
-			(at 87.63 102.87 0)
+			(at 87.63 101.6 0)
 			(hide yes)
 			(show_name no)
@@
 		)
 		(property "Value" "GND"
-			(at 87.63 100.33 0)
+			(at 87.884 99.314 0)
 			(show_name no)
 			(do_not_autoplace no)
@@
 		)
 		(property "Footprint" ""
-			(at 87.63 96.52 0)
+			(at 87.63 95.25 0)
 			(hide yes)
 			(show_name no)
@@
 		)
 		(property "Datasheet" ""
-			(at 87.63 96.52 0)
+			(at 87.63 95.25 0)
 			(hide yes)
 			(show_name no)
@@
 		)
 		(property "Description" "Power symbol creates a global label with name \"GND\" , ground"
-			(at 87.63 96.52 0)
+			(at 87.63 95.25 0)
 			(hide yes)
 			(show_name no)
@@
 	)
 	(symbol
-		(lib_id "S_switches_rotary:1-1825013-0")
-		(at 78.74 93.98 0)
-		(mirror y)
+		(lib_id "TP_testpoints:TP_SMD_2MM")
+		(at 48.26 93.98 0)
 		(unit 1)
 		(body_style 1)
 		(exclude_from_sim no)
-		(in_bom yes)
+		(in_bom no)
 		(on_board yes)
 		(in_pos_files yes)
 		(dnp no)
-		(property "Reference" "S2"
-			(at 80.264 81.788 0)
+		(property "Reference" "TP15"
+			(at 48.26 88.646 0)
 			(show_name no)
 			(do_not_autoplace no)
@@
 			)
 		)
-		(property "Value" "1-1825013-0"
-			(at 79.756 101.854 0)
+		(property "Value" ""
+			(at 48.26 93.98 0)
+			(hide yes)
 			(show_name no)
 			(do_not_autoplace no)
 			(effects
 				(font
-					(size 1.016 1.016)
+					(size 1.27 1.27)
 				)
 			)
 		)
-		(property "Footprint" "switches_smd:1-1825013-0"
-			(at 78.486 98.806 0)
+		(property "Footprint" "testpoints:TP_SMD_0.8mm"
+			(at 48.26 93.98 0)
 			(hide yes)
 			(show_name no)
@@
 		)
 		(property "Datasheet" ""
-			(at 78.74 93.98 0)
+			(at 48.26 93.98 0)
 			(hide yes)
 			(show_name no)
@@
 			)
 		)
-		(property "Description" "SWITCH ROTARY DIP BCD 0.4VA 20V"
-			(at 77.47 110.49 0)
+		(property "Description" "SMD round test point, Pad diameter: 2 mm"
+			(at 48.26 93.98 0)
 			(hide yes)
 			(show_name no)
@@
 			)
 		)
-		(property "PARTNO" "1-1825013-0"
-			(at 76.2 107.95 0)
+		(property "LABEL" "[LABEL]"
+			(at 44.704 88.392 0)
 			(hide yes)
 			(show_name no)
@@
 					(size 1.27 1.27)
 				)
+				(justify left)
 			)
 		)
 		(property "VER" "1"
-			(at 81.28 105.41 0)
+			(at 48.26 93.98 0)
 			(hide yes)
 			(show_name no)
@@
 		)
 		(property "REV" "0"
-			(at 76.2 105.41 0)
-			(hide yes)
-			(show_name no)
-			(do_not_autoplace no)
-			(effects
-				(font
-					(size 1.27 1.27)
-				)
-			)
-		)
-		(property "CRITICAL" ""
-			(at 78.74 93.98 0)
+			(at 48.26 93.98 0)
 			(hide yes)
 			(show_name no)
@@
 			)
 		)
-		(property "EXTERNAL" ""
-			(at 78.74 93.98 0)
+		(property "PARTNO" ""
+			(at 48.26 93.98 0)
 			(hide yes)
 			(show_name no)
@@
 			)
 		)
-		(property "MANUFACTURER" "TE Connectivity ALCOSWITCH Switches"
-			(at 78.74 93.98 0)
+		(property "CRITICAL" ""
+			(at 48.26 93.98 0)
 			(hide yes)
 			(show_name no)
@@
 			)
 		)
-		(property "DIGIKEY_PN_CT" "2266-1-1825013-0-ND"
-			(at 78.74 93.98 0)
+		(property "EXTERNAL" ""
+			(at 48.26 93.98 0)
 			(hide yes)
 			(show_name no)
@@
 			)
 		)
-		(pin "8"
-		)
-		(pin "2"
-		)
-		(pin "C1"
-		)
 		(pin "1"
 		)
-		(pin "C2"
-		)
-		(pin "4"
-		)
 		(instances
 			(project "pcb_0222"
 				(path "/9e623ed9-73f2-41e1-a5f3-2ec43260ffe9"
-					(reference "S2")
+					(reference "TP15")
 					(unit 1)
 				)
@@
 	)
 	(symbol
-		(lib_id "TP_testpoints:TP_SMD_2MM")
-		(at 48.26 93.98 0)
+		(lib_id "S_switches_rotary:CD10RM0SB")
+		(at 78.74 93.98 0)
+		(mirror y)
 		(unit 1)
 		(body_style 1)
 		(exclude_from_sim no)
-		(in_bom no)
+		(in_bom yes)
 		(on_board yes)
 		(in_pos_files yes)
 		(dnp no)
-		(property "Reference" "TP15"
-			(at 48.26 88.646 0)
+		(property "Reference" "S2"
+			(at 80.01 82.55 0)
 			(show_name no)
 			(do_not_autoplace no)
@@
 			)
 		)
-		(property "Value" ""
-			(at 48.26 93.98 0)
-			(hide yes)
+		(property "Value" "CD10RM0SB"
+			(at 79.248 102.108 0)
 			(show_name no)
 			(do_not_autoplace no)
@@
 			)
 		)
-		(property "Footprint" "testpoints:TP_SMD_0.8mm"
-			(at 48.26 93.98 0)
+		(property "Footprint" "switches_smd:CD10RM0SB"
+			(at 78.486 98.806 0)
 			(hide yes)
 			(show_name no)
@@
 		)
 		(property "Datasheet" ""
-			(at 48.26 93.98 0)
+			(at 78.74 93.98 0)
 			(hide yes)
 			(show_name no)
@@
 			)
 		)
-		(property "Description" "SMD round test point, Pad diameter: 2 mm"
-			(at 48.26 93.98 0)
+		(property "Description" "Dip Switch BCD 10 Position Surface Mount Rotary for Tool Actuator 0.4VA 20VAC/DC"
+			(at 77.47 110.49 0)
 			(hide yes)
 			(show_name no)
@@
 			)
 		)
-		(property "LABEL" "[LABEL]"
-			(at 44.704 88.392 0)
+		(property "PARTNO" "CD10RM0SB"
+			(at 76.2 107.95 0)
 			(hide yes)
 			(show_name no)
@@
 					(size 1.27 1.27)
 				)
-				(justify left)
 			)
 		)
 		(property "VER" "1"
-			(at 48.26 93.98 0)
+			(at 81.28 105.41 0)
 			(hide yes)
 			(show_name no)
@@
 		)
 		(property "REV" "0"
-			(at 48.26 93.98 0)
+			(at 76.2 105.41 0)
 			(hide yes)
 			(show_name no)
@@
 			)
 		)
-		(property "PARTNO" ""
-			(at 48.26 93.98 0)
+		(property "CRITICAL" ""
+			(at 78.74 93.98 0)
 			(hide yes)
 			(show_name no)
@@
 			)
 		)
-		(property "CRITICAL" ""
-			(at 48.26 93.98 0)
+		(property "EXTERNAL" ""
+			(at 78.74 93.98 0)
 			(hide yes)
 			(show_name no)
@@
 			)
 		)
-		(property "EXTERNAL" ""
-			(at 48.26 93.98 0)
+		(property "MANUFACTURER" "C&K"
+			(at 78.74 93.98 0)
+			(hide yes)
+			(show_name no)
+			(do_not_autoplace no)
+			(effects
+				(font
+					(size 1.27 1.27)
+				)
+			)
+		)
+		(property "DIGIKEY_PN_CT" "CKN6158-ND"
+			(at 78.74 93.98 0)
 			(hide yes)
 			(show_name no)
@@
 			)
 		)
+		(pin "4"
+		)
+		(pin "C2"
+		)
 		(pin "1"
 		)
+		(pin "C1"
+		)
+		(pin "2"
+		)
+		(pin "8"
+		)
 		(instances
 			(project "pcb_0222"
 				(path "/9e623ed9-73f2-41e1-a5f3-2ec43260ffe9"
-					(reference "TP15")
+					(reference "S2")
 					(unit 1)
 				)

Commit message: C5, C7, C12 PARTNO and D1, R7 VALUE and PARTNO changed after preliminary layout review
Parts:
- removed D1: NZH5V1B,115, diodes_smd:SOD-123F, symbol D_diodes_zener:NZH5V1B
- removed R7: 1K, passives_smd:R_2512, symbol R_resistors:R_2512_1K_1%_1W_AEC-Q200
- added D1: BZT52C5V1, diodes_smd:SOD-123F, symbol D_diodes_zener:BZT52C5V1
- added R7: 3.6K, passives_smd:R_1206, symbol R_resistors:R_1206_3.6K_1%_0.25W
- C12, C7: DIGIKEY_PN_CT 445-181658-1-ND -> 445-CGA6P1X7S1N106K250AECT-ND; PARTNO CGA6P1X7R1N106K250AC -> CGA6P1X7S1N106K250AE; TEMP. COEFF. X7R -> X7S
- C15, C3: DIGIKEY_PN_CT 490-7205-1-ND -> 1276-6794-1-ND; MANUFACTURER Murata Electronics -> Samsung Electro-Mechanics; PARTNO GRM188R6YA475KE15D -> CL10A475KL8NRNC
- C5: DIGIKEY_PN_CT 490-GRM188Z71A106MA73JCT-ND -> 4713-GMC10X7R106K10NTCT-ND; MANUFACTURER Murata Electronics -> Cal-Chip Electronics, Inc.; PARTNO GRM188Z71A106MA73J -> GMC10X7R106K10NT; TOLERANCE 20% -> 10%
Connections:
- net GND: now also R7.1
- net VB_IP: now also D1.C
- net at C6.2, Q1.1: now also D1.A, R7.2

Commit message: Ready for First Release - Complete Package
Parts:
- R7: MANUFACTURER (none) -> YAGEO; Manufacturer YAGEO -> (none)
Changed lines of the file:
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@@
 			)
 		)
-		(property "Manufacturer" "YAGEO"
+		(property "MANUFACTURER" "YAGEO"
 			(at 60.96 48.26 0)
 			(hide yes)
