File: pcb_0222/pcb_0222.kicad_pcb (KiCad board)
At the start: 2 copper layers, 80 x 70 mm, 85 parts, among them J1 5442206, J2 SM02B-PASS-TBT, J3 SM02B-PASS-TBT, J4 HEADER_MALE_THT_0.1"_2x1, J5 HEADER_MALE_THT_0.1"_4x1, J6 SM08B-PASS-TBT, J7 TC-2030-IDC, J8 HEADER_MALE_THT_0.1"_4x1, K1 EE2-3NUH, Q1 BSP170PH6327XTSA1, Q2 BC817-16, U1 NZH5V1B,115, U2 LMR54406DBVR, U3 STM32C011F6P6

Commit message: Placement on Review
Parts:
- added C14: 10uF, passives_smd:C_1210_TDK_CGA6_2.8mm_Tall, F.Cu at (185.3, 99.8)
- added J9: SM08B-PASS-TBT, connectors_headers:SM08B-PASS-TBT, F.Cu at (181.3, 98.1)
- moved J2 66.0 mm to (241.6, 138.1), turned to 90 degrees
- moved J3 65.7 mm to (241.5, 125.8), turned to 90 degrees
- moved TP14 55.1 mm to (199.1, 100.8)
- moved TP5 54.6 mm to (231.5, 141.4)
- moved C7 50.9 mm to (234.0, 138.0), turned to -90 degrees
- moved C8 50.7 mm to (234.0, 125.8), turned to -90 degrees
- moved TP6 49.9 mm to (231.5, 129.4), turned to 180 degrees
- moved R16 46.0 mm to (231.5, 138.0), turned to 90 degrees
- moved R17 45.7 mm to (231.5, 125.8), turned to 90 degrees
- moved TP12 44.3 mm to (218.8, 90.7)
- moved R21 40.5 mm to (194.6, 138.9), turned to 180 degrees
- moved J5 37.1 mm to (201.0, 147.8), turned to 180 degrees
- moved TP13 33.7 mm to (219.4, 147.2)
- moved S2 32.4 mm to (225.8, 129.3), turned to -90 degrees
- moved J8 31.4 mm to (201.0, 143.4), turned to 180 degrees
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Connections:
- J1 pad 1: VB -> GND
- J1 pad 2: GND -> VB
- K1 pad 4: unconnected-(K1-COM_1-Pad4) -> Net-(K1-COM_1)
- K1 pad 5: unconnected-(K1-NO_1-Pad5) -> GND

Commit message: SCH review comments fixed
Parts:
- removed the C13 at (211.1, 131.8)
- removed the G*** at (229.6, 115.4)
- removed the G*** at (191.5, 130.7)
- removed the J4 at (199.1, 135.7)
- removed the J5 at (201.0, 147.8)
- removed the R21 at (194.6, 138.9)
- removed the U1 at (225.1, 95.9)
- added C15: 4.7uF, passives_smd:C_0603, F.Cu at (195.7, 125.6)
- added C8: 10nF, passives_smd:C_0603, F.Cu at (214.5, 125.7)
- added D1: NZH5V1B,115, diodes_smd:SOD-123F, F.Cu at (225.1, 95.7)
- added G***: LOGO, LOGO, F.Cu at (193.1, 96.0)
- added J7: HEADER_MALE_THT_0.1"_4x1, connectors_headers:61300411121, F.Cu at (226.1, 124.9)
- added J9: HEADER_MALE_THT_0.1"_4x1, connectors_headers:61300411121, F.Cu at (226.1, 145.3)
- added R14: 10K, passives_smd:R_0603, F.Cu at (214.5, 123.7)
- added R23: 4K7, passives_smd:R_0603, F.Cu at (231.7, 143.7)
- added TP10: ~, testpoints:TP_SMD_0.8mm, F.Cu at (211.7, 123.9)
- added TVS2: 3V3, diodes_smd:2-DFN_(1.6x1), F.Cu at (214.5, 128.0)
- added TVS3: 3V3, diodes_smd:2-DFN_(1.6x1), F.Cu at (233.8, 130.1)
- added TVS4: 3V3, diodes_smd:2-DFN_(1.6x1), F.Cu at (233.9, 116.7)
- added TVS5: USBLC6-2SC6, packages_smd:SOT-23-6 [2.8x2.93x1.1,P=0.95]mm, F.Cu at (193.5, 139.7)
- added TVS6: 3V3, diodes_smd:2-DFN_(1.6x1), F.Cu at (205.7, 140.9)
- added TVS7: USBLC6-2SC6, packages_smd:SOT-23-6 [2.8x2.93x1.1,P=0.95]mm, F.Cu at (221.8, 128.8)
- added TVS8: USBLC6-2SC6, packages_smd:SOT-23-6 [2.8x2.93x1.1,P=0.95]mm, F.Cu at (221.9, 141.7)
- J8: value HEADER_MALE_THT_0.1"_4x1 -> HEADER_MALE_THT_0.1"_2x1; footprint connectors_headers:61300411121 -> connectors_headers:77311-118-02LF
- R5: value 22.1K -> 69.8K
- R9: value 69.8K -> 22.1K
- moved R22 32.0 mm to (231.7, 140.2), turned to 180 degrees
- moved TP4 22.3 mm to (236.8, 140.2)
- moved TP2 17.4 mm to (236.8, 146.3)
- moved C14 16.2 mm to (192.8, 125.6), turned to 90 degrees
- moved R10 14.8 mm to (216.5, 118.8)
- moved R11 14.8 mm to (213.4, 118.8)
- moved R12 14.8 mm to (216.5, 110.7)
- moved R13 14.8 mm to (213.4, 110.7)
- moved TP13 14.8 mm to (216.5, 113.8)
- moved TP15 14.8 mm to (213.4, 115.8)
- moved TP17 14.8 mm to (216.5, 115.8)
- moved TP9 14.8 mm to (213.4, 113.8)
- moved S2 14.7 mm to (222.6, 114.9)
- moved TP14 12.9 mm to (209.4, 149.3)
- moved C13 12.0 mm to (195.7, 129.1), turned to 90 degrees
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- renumbered C8 to C10, C10 to C11, C9 to C12, C11 to C13, C12 to C14, C14 to C7, C7 to C9, D1 to D2, J9 to J4, J7 to J5, R16 to R15, R17 to R16, R14 to R17, R15 to R18, R18 to R20, R20 to R21, TP12 to TP1, TP5 to TP11, TP6 to TP12, TP8 to TP13, TP7 to TP14, TP10 to TP15, TP9 to TP16, TP11 to TP17, TP16 to TP18, TP17 to TP19, TP13 to TP2, TP14 to TP3, TP15 to TP4, TP1 to TP5, TP2 to TP6, TP3 to TP7, TP18 to TP8, TP4 to TP9, U2 to U1, U3 to U2
Connections:
- J5 pad 2: /SWDIO -> Net-(J5-SWDIO)
- J5 pad 3: /SWCLK -> Net-(J5-SWCLK)
- J8 pad 2: /SDA1 -> /SWCLK
- PB1 pad 1: GND -> /MCU_TEST
- PB1 pad 2: GND -> /MCU_TEST
- PB1 pad 3: /NRST -> GND
- PB1 pad 4: /NRST -> GND
- U2 pad 15: unconnected-(U3-PA8-Pad15) -> /MCU_TEST

Commit message: working on Layout
Parts:
- J1: value 5442206 -> S2P-VH; footprint connectors_terminal_blocks:5442206 -> connectors_headers:S2P-VH
- moved G*** 44.0 mm to (186.1, 139.5)
- moved J1 8.33 mm to (233.3, 107.0)
- moved R7 7.95 mm to (221.8, 92.3)
- moved C6 7.91 mm to (217.4, 89.8)
- moved D1 7.84 mm to (217.4, 94.5)
- moved R8 7.81 mm to (204.5, 102.8)
- moved M4 7.79 mm to (244.2, 147.8)
- moved TP8 7.44 mm to (208.1, 102.8)
- moved R4 7.44 mm to (208.1, 100.4)
- moved LED2 7.31 mm to (196.5, 89.9)
- moved LED1 7.24 mm to (210.3, 103.9)
- moved TP7 7.20 mm to (197.7, 95.9)
- moved C4 7.18 mm to (213.9, 95.2)
- moved C2 7.18 mm to (200.0, 99.9)
- moved R3 7.18 mm to (213.9, 103.1)
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Routing:
- added copper zone on F.Cu, net Net-(C6-Pad2)
- added copper zone on F.Cu, net Net-(F1-Pad1)
- added copper zone on B.Cu, net VB
- added copper zone on F.Cu, net VB
- added copper zone on F.Cu, net VB_IP

Commit message: Layout Ready for Review
Parts:
- moved LED1 16.9 mm to (217.9, 88.7), turned to 180 degrees
- moved C11 15.1 mm to (190.9, 140.3), turned to -90 degrees
- moved G*** 12.5 mm to (190.5, 127.7)
- moved J8 12.4 mm to (205.3, 146.8), turned to 180 degrees
- moved R3 12.1 mm to (215.1, 91.0), turned to -90 degrees
- moved TP19 12.0 mm to (198.4, 121.2)
- moved R14 11.9 mm to (216.9, 135.3), turned to -90 degrees
- moved R23 11.6 mm to (221.5, 138.3)
- moved TVS5 11.4 mm to (204.6, 142.2)
- moved R22 11.2 mm to (221.5, 144.7), turned to 0 degrees
- moved TVS6 9.71 mm to (197.9, 135.6), turned to 180 degrees
- moved C8 9.67 mm to (215.0, 135.4), turned to 90 degrees
- moved TP10 9.16 mm to (212.8, 132.6), turned to 180 degrees
- moved J7 8.00 mm to (226.1, 132.9), turned to 90 degrees
- moved R21 7.70 mm to (201.9, 121.2), turned to 0 degrees
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Routing:
- net /MCU_SW2: track 0.00 -> 50.8 mm, vias 0 -> 4
- net /MCU_BCD0: track 0.00 -> 48.0 mm, vias 0 -> 3
- net +3V3: track 0.00 -> 41.9 mm, vias 0 -> 22
- net /SWCLK: track 0.00 -> 40.9 mm, vias 0 -> 3
- net /SCL1: track 0.00 -> 40.8 mm, vias 0 -> 2
- net /MCU_SW1: track 0.00 -> 39.1 mm, vias 0 -> 4
- net /SDA1: track 0.00 -> 33.9 mm, vias 0 -> 2
- net /MCU_BCD3: track 0.00 -> 33.7 mm, vias 0 -> 4
- net /MCU_DIP1: track 0.00 -> 31.9 mm, vias 0 -> 2
- net /MCU_BCD1: track 0.00 -> 31.8 mm, vias 0 -> 2
- net /MCU_BCD2: track 0.00 -> 31.5 mm, vias 0 -> 2
- net /MCU_LED: track 0.00 -> 27.6 mm, vias 0 -> 4
- net /SWDIO: track 0.00 -> 23.0 mm, vias 0 -> 2
- net Net-(J5-SWDIO): track 0.00 -> 21.0 mm, vias 0 -> 2
- net /MCU_DIP2: track 0.00 -> 20.0 mm
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- added copper zone on B.Cu, net +3V3
- added copper zone on F.Cu, net +3V3
- added copper zone on F.Cu, net /FB
- added copper zone on F.Cu, net /MCU_DIP1
- added copper zone on F.Cu, net /MCU_DIP2
- added copper zone on F.Cu, net /MCU_RELAY
- added copper zone on F.Cu, net /MCU_SW1
- added copper zone on F.Cu, net /MCU_SW2
- added copper zone on F.Cu, net /MCU_TEST
- added copper zone on F.Cu, net /NRST
- added copper zone on F.Cu, net /SW
- added copper zone on B.Cu, net GND
- added copper zone on F.Cu, net GND
- added copper zone on F.Cu, net Net-(C2-Pad2)
- added copper zone on F.Cu, net Net-(K1-COIL-)
- added copper zone on F.Cu, net Net-(K1-COM_1)
- added copper zone on F.Cu, net Net-(K1-COM_2)
- added copper zone on F.Cu, net Net-(LED1-PadA)
- added copper zone on F.Cu, net Net-(U1-CB)
- added copper zone on F.Cu, net Net-(U1-EN)
- added copper zone on F.Cu, net Net-(U1-VIN)
- added copper zone on B.Cu, net VB_IP
Other:
- rule pad_to_mask_clearance: 0.1 -> 0.05
- rule solder_mask_min_width: 0.2 -> 0.05

Commit message: Layout Review Pending + Preliminary Manufacturer Package Generated
Parts:
- removed the G*** at (324.4, 259.8)
- moved C1 57.2 mm to (149.0, 82.0)
- moved C10 57.2 mm to (176.4, 103.7)
- moved C11 57.2 mm to (135.7, 125.3)
- moved C12 57.2 mm to (130.0, 111.7)
- moved C13 57.2 mm to (141.9, 116.3)
- moved C14 57.2 mm to (140.0, 112.5)
- moved C15 57.2 mm to (141.9, 112.5)
- moved C3 57.2 mm to (155.8, 84.3)
- moved C4 57.2 mm to (153.5, 84.3)
- moved C6 57.2 mm to (162.8, 77.3)
- moved C7 57.2 mm to (130.0, 84.8)
- moved C9 57.2 mm to (176.3, 115.9)
- moved D1 57.2 mm to (161.1, 80.9)
- moved D2 57.2 mm to (148.3, 98.5)
- moved G*** 57.2 mm to (135.2, 112.7)
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Other:
- board text added: "R7"
- board text added: "TVS1"

Commit message: Board characteristics add into F.Fab and ASM DWG + UID add into Silkscreen Layer
Parts:
- removed the G*** at (135.2, 112.7)
- added G***: LOGO, LOGO, F.Cu at (135.6, 111.7)
- added G***: LOGO, LOGO, F.Cu at (199.5, 172.7)
Other:
- rule pad_to_mask_clearance: 0.05 -> 0.0508
- rule solder_mask_min_width: 0.05 -> 0.0508
- board text added: "UV Unit LR0203-0000"
